Commit message: Added xacro files for gazebo

File: urdf/canadarm2.urdf.xacro (robot description, xacro)
@@ -1,4 +1,4 @@
 <?xml version="1.0"?>
-<robot name="dextre" xmlns:xacro="http://www.ros.org/wiki/xacro">
+<robot name="canadarm2" xmlns:xacro="http://www.ros.org/wiki/xacro">
   <!-- CANADARM2 -->
   <xacro:macro name="canadarm2" params=" parent:='' ">
@@ -22,7 +22,4 @@
        <mesh filename="package://iss_description/meshes/canadarm2_base.dae" scale="1 1 1"/>
      </geometry>
-     <material name="Cyan">
-       <color rgba="0 1.0 1.0 1.0"/>
-     </material>
    </visual>
    <collision>
@@ -45,7 +42,4 @@
         <mesh filename="package://iss_description/meshes/canadarm2_link_1.dae" scale="1 1 1"/>
       </geometry>
-      <material name="Cyan">
-        <color rgba="0 1.0 1.0 1.0"/>
-      </material>
     </visual>
     <collision>
@@ -68,7 +62,4 @@
         <mesh filename="package://iss_description/meshes/canadarm2_link_2.dae" scale="1 1 1"/>
       </geometry>
-      <material name="Cyan">
-        <color rgba="0 1.0 1.0 1.0"/>
-      </material>
     </visual>
     <collision>
@@ -91,7 +82,4 @@
         <mesh filename="package://iss_description/meshes/canadarm2_link_3.dae" scale="1 1 1"/>
       </geometry>
-      <material name="Cyan">
-        <color rgba="0 1.0 1.0 1.0"/>
-      </material>
     </visual>
     <collision>
@@ -114,7 +102,4 @@
         <mesh filename="package://iss_description/meshes/canadarm2_link_4.dae" scale="1 1 1"/>
       </geometry>
-      <material name="Cyan">
-        <color rgba="0 1.0 1.0 1.0"/>
-      </material>
     </visual>
     <collision>
@@ -137,7 +122,4 @@
         <mesh filename="package://iss_description/meshes/canadarm2_link_5.dae" scale="1 1 1"/>
       </geometry>
-      <material name="Cyan">
-        <color rgba="0 1.0 1.0 1.0"/>
-      </material>
     </visual>
     <collision>
@@ -160,7 +142,4 @@
         <mesh filename="package://iss_description/meshes/canadarm2_link_6.dae" scale="1 1 1"/>
       </geometry>
-      <material name="Cyan">
-        <color rgba="0 1.0 1.0 1.0"/>
-      </material>
     </visual>
     <collision>
@@ -183,7 +162,4 @@
         <mesh filename="package://iss_description/meshes/canadarm2_link_7.dae" scale="1 1 1"/>
       </geometry>
-      <material name="Cyan">
-        <color rgba="0 1.0 1.0 1.0"/>
-      </material>
     </visual>
     <collision>

File: urdf/dextre.urdf.xacro (robot description, xacro)
@@ -15,7 +15,4 @@
        <mesh filename="package://iss_description/meshes/dextre_base.dae" scale="1 1 1"/>
      </geometry>
-     <material name="Cyan">
-       <color rgba="0 1.0 1.0 1.0"/>
-     </material>
    </visual>
    <collision>
@@ -38,7 +35,4 @@
        <mesh filename="package://iss_description/meshes/dextre_body.dae" scale="1 1 1"/>
      </geometry>
-     <material name="Cyan">
-       <color rgba="0 1.0 1.0 1.0"/>
-     </material>
    </visual>
    <collision>
@@ -61,7 +55,4 @@
        <mesh filename="package://iss_description/meshes/dextre_tool_platform.dae" scale="1 1 1"/>
      </geometry>
-     <material name="Cyan">
-       <color rgba="0 1.0 1.0 1.0"/>
-     </material>
    </visual>
    <collision>
@@ -84,7 +75,4 @@
        <mesh filename="package://iss_description/meshes/dextre_latching_end_effector.dae" scale="1 1 1"/>
      </geometry>
-     <material name="Cyan">
-       <color rgba="0 1.0 1.0 1.0"/>
-     </material>
    </visual>
    <collision>
@@ -139,7 +127,4 @@
        <mesh filename="package://iss_description/meshes/dextre_arm_1_shoulder_roll.dae" scale="1 1 1"/>
      </geometry>
-     <material name="Cyan">
-       <color rgba="0 1.0 1.0 1.0"/>
-     </material>
    </visual>
    <collision>
@@ -162,7 +147,4 @@
        <mesh filename="package://iss_description/meshes/dextre_arm_1_shoulder_yaw.dae" scale="1 1 1"/>
      </geometry>
-     <material name="Cyan">
-       <color rgba="0 1.0 1.0 1.0"/>
-     </material>
    </visual>
    <collision>
@@ -185,7 +167,4 @@
        <mesh filename="package://iss_description/meshes/dextre_arm_1_shoulder_pitch.dae" scale="1 1 1"/>
      </geometry>
-     <material name="Cyan">
-       <color rgba="0 1.0 1.0 1.0"/>
-     </material>
    </visual>
    <collision>
@@ -208,7 +187,4 @@
        <mesh filename="package://iss_description/meshes/dextre_arm_1_elbow_pitch.dae" scale="1 1 1"/>
      </geometry>
-     <material name="Cyan">
-       <color rgba="0 1.0 1.0 1.0"/>
-     </material>
    </visual>
    <collision>
@@ -231,7 +207,4 @@
        <mesh filename="package://iss_description/meshes/dextre_arm_1_wrist_pitch_yaw.dae" scale="1 1 1"/>
      </geometry>
-     <material name="Cyan">
-       <color rgba="0 1.0 1.0 1.0"/>
-     </material>
    </visual>
    <collision>
@@ -254,7 +227,4 @@
        <mesh filename="package://iss_description/meshes/dextre_arm_1_wrist_roll.dae" scale="1 1 1"/>
      </geometry>
-     <material name="Cyan">
-       <color rgba="0 1.0 1.0 1.0"/>
-     </material>
    </visual>
    <collision>
@@ -331,7 +301,4 @@
        <mesh filename="package://iss_description/meshes/dextre_arm_2_shoulder_roll.dae" scale="1 1 1"/>
      </geometry>
-     <material name="Cyan">
-       <color rgba="0 1.0 1.0 1.0"/>
-     </material>
    </visual>
    <collision>
@@ -354,7 +321,4 @@
        <mesh filename="package://iss_description/meshes/dextre_arm_2_shoulder_yaw.dae" scale="1 1 1"/>
      </geometry>
-     <material name="Cyan">
-       <color rgba="0 1.0 1.0 1.0"/>
-     </material>
    </visual>
    <collision>
@@ -377,7 +341,4 @@
        <mesh filename="package://iss_description/meshes/dextre_arm_2_shoulder_pitch.dae" scale="1 1 1"/>
      </geometry>
-     <material name="Cyan">
-       <color rgba="0 1.0 1.0 1.0"/>
-     </material>
    </visual>
    <collision>
@@ -400,7 +361,4 @@
        <mesh filename="package://iss_description/meshes/dextre_arm_2_elbow_pitch.dae" scale="1 1 1"/>
      </geometry>
-     <material name="Cyan">
-       <color rgba="0 1.0 1.0 1.0"/>
-     </material>
    </visual>
    <collision>
@@ -423,7 +381,4 @@
        <mesh filename="package://iss_description/meshes/dextre_arm_2_wrist_pitch_yaw.dae" scale="1 1 1"/>
      </geometry>
-     <material name="Cyan">
-       <color rgba="0 1.0 1.0 1.0"/>
-     </material>
    </visual>
    <collision>
@@ -446,7 +401,4 @@
        <mesh filename="package://iss_description/meshes/dextre_arm_2_wrist_roll.dae" scale="1 1 1"/>
      </geometry>
-     <material name="Cyan">
-       <color rgba="0 1.0 1.0 1.0"/>
-     </material>
    </visual>
    <collision>

File: urdf/mobile_base_system.urdf.xacro (robot description, xacro)
@@ -1,7 +1,6 @@
 <?xml version="1.0"?>
-<robot name="mobile_servicing_system" xmlns:xacro="http://www.ros.org/wiki/xacro">
-  <xacro:include filename="$(find iss_description)/urdf/canadarm2.urdf.xacro"/>
-  <xacro:include filename="$(find iss_description)/urdf/dextre.urdf.xacro"/>
-  <link name="world"/>
+<robot name="mobile_base_system" xmlns:xacro="http://www.ros.org/wiki/xacro">
+  <!-- MOBILE BASE SYSTEM -->
+  <xacro:macro name="mobile_base_system" params=" parent:='world' ">
   <link name="body">
    <inertial>
@@ -15,7 +14,4 @@
        <mesh filename="package://iss_description/meshes/iss_stationary.dae" scale="1 1 1"/>
      </geometry>
-     <material name="Cyan">
-       <color rgba="0 1.0 1.0 1.0"/>
-     </material>
    </visual>
    <collision>
@@ -38,7 +34,4 @@
        <mesh filename="package://iss_description/meshes/mobile_base_system.dae" scale="1 1 1"/>
      </geometry>
-     <material name="Cyan">
-       <color rgba="0 1.0 1.0 1.0"/>
-     </material>
    </visual>
    <collision>
@@ -54,5 +47,5 @@
   <joint name="joint_world" type="fixed">
       <origin rpy="0 0 0" xyz="0 0 0"/>
-      <parent link="world"/>
+      <parent link="${parent}"/>
       <child link="body"/>
   </joint>
@@ -80,5 +73,4 @@
       <limit effort="1000.0" lower="-15.0" upper="42.0" velocity="0.5"/>
   </joint>
-  <xacro:dextre parent="canadarm2_link_7"/>
-  <xacro:canadarm2 parent="mobile_base_system"/>
+  </xacro:macro>
 </robot>
