Commit message: Reorganized files and added mobility for Solar Panels

File: urdf/canadarm2.urdf.xacro (robot description, xacro)
@@ -20,5 +20,5 @@
      <origin xyz="0 0 0" rpy="0.35691983 0.0 0.572468" />
      <geometry>
-       <mesh filename="package://iss_description/meshes/canadarm2_base.dae" scale="1 1 1"/>
+       <mesh filename="package://iss_description/meshes/canadarm2/base.dae" scale="1 1 1"/>
      </geometry>
    </visual>
@@ -26,5 +26,5 @@
      <origin xyz="0 0 0" rpy="0 0 0"/>
      <geometry>
-       <mesh filename="package://iss_description/meshes/canadarm2_base.dae" scale="1 1 1"/>
+       <mesh filename="package://iss_description/meshes/canadarm2/base.dae" scale="1 1 1"/>
      </geometry>
    </collision>
@@ -40,5 +40,5 @@
       <origin xyz="0 0 0" rpy="0.0 -0.488692 0.663225" /> <!-- Blender: 0 -28 38-->
       <geometry>
-        <mesh filename="package://iss_description/meshes/canadarm2_link_1.dae" scale="1 1 1"/>
+        <mesh filename="package://iss_description/meshes/canadarm2/link_1.dae" scale="1 1 1"/>
       </geometry>
     </visual>
@@ -46,5 +46,5 @@
       <origin xyz="0 0 0" rpy="0.0 -0.488692 0.663225"/>
       <geometry>
-        <mesh filename="package://iss_description/meshes/canadarm2_link_1.dae" scale="1 1 1"/>
+        <mesh filename="package://iss_description/meshes/canadarm2/link_1.dae" scale="1 1 1"/>
       </geometry>
     </collision>
@@ -60,5 +60,5 @@
       <origin xyz="0 0 0" rpy="0 -0.49131018 0" /> <!-- Blender: 0.0 -28.15 0.0-->
       <geometry>
-        <mesh filename="package://iss_description/meshes/canadarm2_link_2.dae" scale="1 1 1"/>
+        <mesh filename="package://iss_description/meshes/canadarm2/link_2.dae" scale="1 1 1"/>
       </geometry>
     </visual>
@@ -66,5 +66,5 @@
       <origin xyz="0 0 0" rpy="0 -0.49131018 0"/>
       <geometry>
-        <mesh filename="package://iss_description/meshes/canadarm2_link_2.dae" scale="1 1 1"/>
+        <mesh filename="package://iss_description/meshes/canadarm2/link_2.dae" scale="1 1 1"/>
       </geometry>
     </collision>
@@ -80,11 +80,11 @@
       <origin xyz="0 0 0" rpy="0 0 0" />
       <geometry>
-        <mesh filename="package://iss_description/meshes/canadarm2_link_3.dae" scale="1 1 1"/>
-      </geometry>
-    </visual>
-    <collision>
-      <origin xyz="0 0 0" rpy="0 0 0"/>
-      <geometry>
-        <mesh filename="package://iss_description/meshes/canadarm2_link_3.dae" scale="1 1 1"/>
+        <mesh filename="package://iss_description/meshes/canadarm2/link_3.dae" scale="1 1 1"/>
+      </geometry>
+    </visual>
+    <collision>
+      <origin xyz="0 0 0" rpy="0 0 0"/>
+      <geometry>
+        <mesh filename="package://iss_description/meshes/canadarm2/link_3.dae" scale="1 1 1"/>
       </geometry>
     </collision>
@@ -100,11 +100,11 @@
       <origin xyz="0 0 0" rpy="0 0 0" />
       <geometry>
-        <mesh filename="package://iss_description/meshes/canadarm2_link_4.dae" scale="1 1 1"/>
-      </geometry>
-    </visual>
-    <collision>
-      <origin xyz="0 0 0" rpy="0 0 0"/>
-      <geometry>
-        <mesh filename="package://iss_description/meshes/canadarm2_link_4.dae" scale="1 1 1"/>
+        <mesh filename="package://iss_description/meshes/canadarm2/link_4.dae" scale="1 1 1"/>
+      </geometry>
+    </visual>
+    <collision>
+      <origin xyz="0 0 0" rpy="0 0 0"/>
+      <geometry>
+        <mesh filename="package://iss_description/meshes/canadarm2/link_4.dae" scale="1 1 1"/>
       </geometry>
     </collision>
@@ -120,11 +120,11 @@
       <origin xyz="0 0 0" rpy="0 0 0" />
       <geometry>
-        <mesh filename="package://iss_description/meshes/canadarm2_link_5.dae" scale="1 1 1"/>
-      </geometry>
-    </visual>
-    <collision>
-      <origin xyz="0 0 0" rpy="0 0 0"/>
-      <geometry>
-        <mesh filename="package://iss_description/meshes/canadarm2_link_5.dae" scale="1 1 1"/>
+        <mesh filename="package://iss_description/meshes/canadarm2/link_5.dae" scale="1 1 1"/>
+      </geometry>
+    </visual>
+    <collision>
+      <origin xyz="0 0 0" rpy="0 0 0"/>
+      <geometry>
+        <mesh filename="package://iss_description/meshes/canadarm2/link_5.dae" scale="1 1 1"/>
       </geometry>
     </collision>
@@ -140,11 +140,11 @@
       <origin xyz="0 0 0" rpy="0 0 0" />
       <geometry>
-        <mesh filename="package://iss_description/meshes/canadarm2_link_6.dae" scale="1 1 1"/>
-      </geometry>
-    </visual>
-    <collision>
-      <origin xyz="0 0 0" rpy="0 0 0"/>
-      <geometry>
-        <mesh filename="package://iss_description/meshes/canadarm2_link_6.dae" scale="1 1 1"/>
+        <mesh filename="package://iss_description/meshes/canadarm2/link_6.dae" scale="1 1 1"/>
+      </geometry>
+    </visual>
+    <collision>
+      <origin xyz="0 0 0" rpy="0 0 0"/>
+      <geometry>
+        <mesh filename="package://iss_description/meshes/canadarm2/link_6.dae" scale="1 1 1"/>
       </geometry>
     </collision>
@@ -160,11 +160,11 @@
       <origin xyz="0 0 0" rpy="0 0 0" />
       <geometry>
-        <mesh filename="package://iss_description/meshes/canadarm2_link_7.dae" scale="1 1 1"/>
-      </geometry>
-    </visual>
-    <collision>
-      <origin xyz="0 0 0" rpy="0 0 0"/>
-      <geometry>
-        <mesh filename="package://iss_description/meshes/canadarm2_link_7.dae" scale="1 1 1"/>
+        <mesh filename="package://iss_description/meshes/canadarm2/link_7.dae" scale="1 1 1"/>
+      </geometry>
+    </visual>
+    <collision>
+      <origin xyz="0 0 0" rpy="0 0 0"/>
+      <geometry>
+        <mesh filename="package://iss_description/meshes/canadarm2/link_7.dae" scale="1 1 1"/>
       </geometry>
     </collision>

File: urdf/dextre.urdf.xacro (robot description, xacro)
@@ -13,11 +13,11 @@
      <origin xyz="0 0 0" rpy="0 0 0" />
      <geometry>
-       <mesh filename="package://iss_description/meshes/dextre_base.dae" scale="1 1 1"/>
-     </geometry>
-   </visual>
-   <collision>
-     <origin xyz="0 0 0" rpy="0 0 0"/>
-     <geometry>
-       <mesh filename="package://iss_description/meshes/dextre_base.dae" scale="1 1 1"/>
+       <mesh filename="package://iss_description/meshes/dextre/base.dae" scale="1 1 1"/>
+     </geometry>
+   </visual>
+   <collision>
+     <origin xyz="0 0 0" rpy="0 0 0"/>
+     <geometry>
+       <mesh filename="package://iss_description/meshes/dextre/base.dae" scale="1 1 1"/>
      </geometry>
    </collision>
@@ -33,11 +33,11 @@
      <origin xyz="0 0 0" rpy="0 0 0" />
      <geometry>
-       <mesh filename="package://iss_description/meshes/dextre_body.dae" scale="1 1 1"/>
-     </geometry>
-   </visual>
-   <collision>
-     <origin xyz="0 0 0" rpy="0 0 0"/>
-     <geometry>
-       <mesh filename="package://iss_description/meshes/dextre_body.dae" scale="1 1 1"/>
+       <mesh filename="package://iss_description/meshes/dextre/body.dae" scale="1 1 1"/>
+     </geometry>
+   </visual>
+   <collision>
+     <origin xyz="0 0 0" rpy="0 0 0"/>
+     <geometry>
+       <mesh filename="package://iss_description/meshes/dextre/body.dae" scale="1 1 1"/>
      </geometry>
    </collision>
@@ -53,11 +53,11 @@
      <origin xyz="0 0 0" rpy="0 0 0" />
      <geometry>
-       <mesh filename="package://iss_description/meshes/dextre_tool_platform.dae" scale="1 1 1"/>
-     </geometry>
-   </visual>
-   <collision>
-     <origin xyz="0 0 0" rpy="0 0 0"/>
-     <geometry>
-       <mesh filename="package://iss_description/meshes/dextre_tool_platform.dae" scale="1 1 1"/>
+       <mesh filename="package://iss_description/meshes/dextre/tool_platform.dae" scale="1 1 1"/>
+     </geometry>
+   </visual>
+   <collision>
+     <origin xyz="0 0 0" rpy="0 0 0"/>
+     <geometry>
+       <mesh filename="package://iss_description/meshes/dextre/tool_platform.dae" scale="1 1 1"/>
      </geometry>
    </collision>
@@ -73,11 +73,11 @@
      <origin xyz="0 0 0" rpy="0 0 0" />
      <geometry>
-       <mesh filename="package://iss_description/meshes/dextre_latching_end_effector.dae" scale="1 1 1"/>
-     </geometry>
-   </visual>
-   <collision>
-     <origin xyz="0 0 0" rpy="0 0 0"/>
-     <geometry>
-       <mesh filename="package://iss_description/meshes/dextre_latching_end_effector.dae" scale="1 1 1"/>
+       <mesh filename="package://iss_description/meshes/dextre/latching_end_effector.dae" scale="1 1 1"/>
+     </geometry>
+   </visual>
+   <collision>
+     <origin xyz="0 0 0" rpy="0 0 0"/>
+     <geometry>
+       <mesh filename="package://iss_description/meshes/dextre/latching_end_effector.dae" scale="1 1 1"/>
      </geometry>
    </collision>
@@ -125,5 +125,5 @@
      <origin xyz="0 0 0" rpy="0 0.785398 0" />
      <geometry>
-       <mesh filename="package://iss_description/meshes/dextre_arm_1_shoulder_roll.dae" scale="1 1 1"/>
+       <mesh filename="package://iss_description/meshes/dextre/arm_1/shoulder_roll.dae" scale="1 1 1"/>
      </geometry>
    </visual>
@@ -131,5 +131,5 @@
      <origin xyz="0 0 0" rpy="0 0.785398 0"/>
      <geometry>
-       <mesh filename="package://iss_description/meshes/dextre_arm_1_shoulder_roll.dae" scale="1 1 1"/>
+       <mesh filename="package://iss_description/meshes/dextre/arm_1/shoulder_roll.dae" scale="1 1 1"/>
      </geometry>
    </collision>
@@ -145,5 +145,5 @@
      <origin xyz="0 0 0" rpy="0 0.7941248 0" /> <!-- 0.0 -45.5 0.0-->
      <geometry>
-       <mesh filename="package://iss_description/meshes/dextre_arm_1_shoulder_yaw.dae" scale="1 1 1"/>
+       <mesh filename="package://iss_description/meshes/dextre/arm_1/shoulder_yaw.dae" scale="1 1 1"/>
      </geometry>
    </visual>
@@ -151,5 +151,5 @@
      <origin xyz="0 0 0" rpy="0 0.7941248 0"/>
      <geometry>
-       <mesh filename="package://iss_description/meshes/dextre_arm_1_shoulder_yaw.dae" scale="1 1 1"/>
+       <mesh filename="package://iss_description/meshes/dextre/arm_1/shoulder_yaw.dae" scale="1 1 1"/>
      </geometry>
    </collision>
@@ -165,11 +165,11 @@
      <origin xyz="0 0 0" rpy="0 0 0" />
      <geometry>
-       <mesh filename="package://iss_description/meshes/dextre_arm_1_shoulder_pitch.dae" scale="1 1 1"/>
-     </geometry>
-   </visual>
-   <collision>
-     <origin xyz="0 0 0" rpy="0 0 0"/>
-     <geometry>
-       <mesh filename="package://iss_description/meshes/dextre_arm_1_shoulder_pitch.dae" scale="1 1 1"/>
+       <mesh filename="package://iss_description/meshes/dextre/arm_1/shoulder_pitch.dae" scale="1 1 1"/>
+     </geometry>
+   </visual>
+   <collision>
+     <origin xyz="0 0 0" rpy="0 0 0"/>
+     <geometry>
+       <mesh filename="package://iss_description/meshes/dextre/arm_1/shoulder_pitch.dae" scale="1 1 1"/>
      </geometry>
    </collision>
@@ -185,11 +185,11 @@
      <origin xyz="0 0 0" rpy="0 0 0" />
      <geometry>
-       <mesh filename="package://iss_description/meshes/dextre_arm_1_elbow_pitch.dae" scale="1 1 1"/>
-     </geometry>
-   </visual>
-   <collision>
-     <origin xyz="0 0 0" rpy="0 0 0"/>
-     <geometry>
-       <mesh filename="package://iss_description/meshes/dextre_arm_1_elbow_pitch.dae" scale="1 1 1"/>
+       <mesh filename="package://iss_description/meshes/dextre/arm_1/elbow_pitch.dae" scale="1 1 1"/>
+     </geometry>
+   </visual>
+   <collision>
+     <origin xyz="0 0 0" rpy="0 0 0"/>
+     <geometry>
+       <mesh filename="package://iss_description/meshes/dextre/arm_1/elbow_pitch.dae" scale="1 1 1"/>
      </geometry>
    </collision>
@@ -205,11 +205,11 @@
      <origin xyz="0 0 0" rpy="0 0 0" />
      <geometry>
-       <mesh filename="package://iss_description/meshes/dextre_arm_1_wrist_pitch_yaw.dae" scale="1 1 1"/>
-     </geometry>
-   </visual>
-   <collision>
-     <origin xyz="0 0 0" rpy="0 0 0"/>
-     <geometry>
-       <mesh filename="package://iss_description/meshes/dextre_arm_1_wrist_pitch_yaw.dae" scale="1 1 1"/>
+       <mesh filename="package://iss_description/meshes/dextre/arm_1/wrist_pitch_yaw.dae" scale="1 1 1"/>
+     </geometry>
+   </visual>
+   <collision>
+     <origin xyz="0 0 0" rpy="0 0 0"/>
+     <geometry>
+       <mesh filename="package://iss_description/meshes/dextre/arm_1/wrist_pitch_yaw.dae" scale="1 1 1"/>
      </geometry>
    </collision>
@@ -225,11 +225,11 @@
      <origin xyz="0 0 0" rpy="0 0 0" />
      <geometry>
-       <mesh filename="package://iss_description/meshes/dextre_arm_1_wrist_roll.dae" scale="1 1 1"/>
-     </geometry>
-   </visual>
-   <collision>
-     <origin xyz="0 0 0" rpy="0 0 0"/>
-     <geometry>
-       <mesh filename="package://iss_description/meshes/dextre_arm_1_wrist_roll.dae" scale="1 1 1"/>
+       <mesh filename="package://iss_description/meshes/dextre/arm_1/wrist_roll.dae" scale="1 1 1"/>
+     </geometry>
+   </visual>
+   <collision>
+     <origin xyz="0 0 0" rpy="0 0 0"/>
+     <geometry>
+       <mesh filename="package://iss_description/meshes/dextre/arm_1/wrist_roll.dae" scale="1 1 1"/>
      </geometry>
    </collision>
@@ -299,11 +299,11 @@
      <origin xyz="0 0 0" rpy="0 -0.785398 0" />
      <geometry>
-       <mesh filename="package://iss_description/meshes/dextre_arm_2_shoulder_roll.dae" scale="1 1 1"/>
-     </geometry>
-   </visual>
-   <collision>
-     <origin xyz="0 0 0" rpy="0 0 0"/>
-     <geometry>
-       <mesh filename="package://iss_description/meshes/dextre_arm_2_shoulder_roll.dae" scale="1 1 1"/>
+       <mesh filename="package://iss_description/meshes/dextre/arm_2/shoulder_roll.dae" scale="1 1 1"/>
+     </geometry>
+   </visual>
+   <collision>
+     <origin xyz="0 0 0" rpy="0 0 0"/>
+     <geometry>
+       <mesh filename="package://iss_description/meshes/dextre/arm_2/shoulder_roll.dae" scale="1 1 1"/>
      </geometry>
    </collision>
@@ -319,11 +319,11 @@
      <origin xyz="0 0 0" rpy="0 -0.7941248 0" /> <!-- 0.0 45.5 0.0-->
      <geometry>
-       <mesh filename="package://iss_description/meshes/dextre_arm_2_shoulder_yaw.dae" scale="1 1 1"/>
-     </geometry>
-   </visual>
-   <collision>
-     <origin xyz="0 0 0" rpy="0 0 0"/>
-     <geometry>
-       <mesh filename="package://iss_description/meshes/dextre_arm_2_shoulder_yaw.dae" scale="1 1 1"/>
+       <mesh filename="package://iss_description/meshes/dextre/arm_2/shoulder_yaw.dae" scale="1 1 1"/>
+     </geometry>
+   </visual>
+   <collision>
+     <origin xyz="0 0 0" rpy="0 0 0"/>
+     <geometry>
+       <mesh filename="package://iss_description/meshes/dextre/arm_2/shoulder_yaw.dae" scale="1 1 1"/>
      </geometry>
    </collision>
@@ -339,11 +339,11 @@
      <origin xyz="0 0 0" rpy="0 0 0" />
      <geometry>
-       <mesh filename="package://iss_description/meshes/dextre_arm_2_shoulder_pitch.dae" scale="1 1 1"/>
-     </geometry>
-   </visual>
-   <collision>
-     <origin xyz="0 0 0" rpy="0 0 0"/>
-     <geometry>
-       <mesh filename="package://iss_description/meshes/dextre_arm_2_shoulder_pitch.dae" scale="1 1 1"/>
+       <mesh filename="package://iss_description/meshes/dextre/arm_2/shoulder_pitch.dae" scale="1 1 1"/>
+     </geometry>
+   </visual>
+   <collision>
+     <origin xyz="0 0 0" rpy="0 0 0"/>
+     <geometry>
+       <mesh filename="package://iss_description/meshes/dextre/arm_2/shoulder_pitch.dae" scale="1 1 1"/>
      </geometry>
    </collision>
@@ -359,11 +359,11 @@
      <origin xyz="0 0 0" rpy="0 0 0" />
      <geometry>
-       <mesh filename="package://iss_description/meshes/dextre_arm_2_elbow_pitch.dae" scale="1 1 1"/>
-     </geometry>
-   </visual>
-   <collision>
-     <origin xyz="0 0 0" rpy="0 0 0"/>
-     <geometry>
-       <mesh filename="package://iss_description/meshes/dextre_arm_2_elbow_pitch.dae" scale="1 1 1"/>
+       <mesh filename="package://iss_description/meshes/dextre/arm_2/elbow_pitch.dae" scale="1 1 1"/>
+     </geometry>
+   </visual>
+   <collision>
+     <origin xyz="0 0 0" rpy="0 0 0"/>
+     <geometry>
+       <mesh filename="package://iss_description/meshes/dextre/arm_2/elbow_pitch.dae" scale="1 1 1"/>
      </geometry>
    </collision>
@@ -379,11 +379,11 @@
      <origin xyz="0 0 0" rpy="0 0 0" />
      <geometry>
-       <mesh filename="package://iss_description/meshes/dextre_arm_2_wrist_pitch_yaw.dae" scale="1 1 1"/>
-     </geometry>
-   </visual>
-   <collision>
-     <origin xyz="0 0 0" rpy="0 0 0"/>
-     <geometry>
-       <mesh filename="package://iss_description/meshes/dextre_arm_2_wrist_pitch_yaw.dae" scale="1 1 1"/>
+       <mesh filename="package://iss_description/meshes/dextre/arm_2/wrist_pitch_yaw.dae" scale="1 1 1"/>
+     </geometry>
+   </visual>
+   <collision>
+     <origin xyz="0 0 0" rpy="0 0 0"/>
+     <geometry>
+       <mesh filename="package://iss_description/meshes/dextre/arm_2/wrist_pitch_yaw.dae" scale="1 1 1"/>
      </geometry>
    </collision>
@@ -399,11 +399,11 @@
      <origin xyz="0 0 0" rpy="0 0 0" />
      <geometry>
-       <mesh filename="package://iss_description/meshes/dextre_arm_2_wrist_roll.dae" scale="1 1 1"/>
-     </geometry>
-   </visual>
-   <collision>
-     <origin xyz="0 0 0" rpy="0 0 0"/>
-     <geometry>
-       <mesh filename="package://iss_description/meshes/dextre_arm_2_wrist_roll.dae" scale="1 1 1"/>
+       <mesh filename="package://iss_description/meshes/dextre/arm_2/wrist_roll.dae" scale="1 1 1"/>
+     </geometry>
+   </visual>
+   <collision>
+     <origin xyz="0 0 0" rpy="0 0 0"/>
+     <geometry>
+       <mesh filename="package://iss_description/meshes/dextre/arm_2/wrist_roll.dae" scale="1 1 1"/>
      </geometry>
    </collision>
