Commit message: increase joint limits to ensure fast demo

File: urdf/canadarm2.urdf.xacro (robot description, xacro)
@@ -178,5 +178,5 @@
       <child link="canadarm2_link_1"/>
       <axis xyz="0 1 0"/>
-      <limit effort="10000.0" lower="-3.1416" upper="3.1416" velocity="0.04"/>
+      <limit effort="100000.0" lower="-3.1416" upper="3.1416" velocity="1.0"/>
   </joint>
   <joint name="joint_canadarm2_2" type="revolute">
@@ -185,5 +185,5 @@
       <child link="canadarm2_link_2"/>
       <axis xyz="0 0 1"/>
-      <limit effort="10000.0" lower="-3.1416" upper="3.1416" velocity="0.04"/>
+      <limit effort="100000.0" lower="-3.1416" upper="3.1416" velocity="1.0"/>
   </joint>
   <joint name="joint_canadarm2_3" type="revolute">
@@ -192,5 +192,5 @@
       <child link="canadarm2_link_3"/>
       <axis xyz="0 1 0"/>
-      <limit effort="10000.0" lower="-3.1416" upper="3.1416" velocity="0.04"/>
+      <limit effort="100000.0" lower="-3.1416" upper="3.1416" velocity="1.0"/>
   </joint>
   <joint name="joint_canadarm2_4" type="revolute">
@@ -199,5 +199,5 @@
       <child link="canadarm2_link_4"/>
       <axis xyz="0 1 0"/>
-      <limit effort="10000.0" lower="-3.1416" upper="3.1416" velocity="0.04"/>
+      <limit effort="100000.0" lower="-3.1416" upper="3.1416" velocity="1.0"/>
   </joint>
   <joint name="joint_canadarm2_5" type="revolute">
@@ -206,5 +206,5 @@
       <child link="canadarm2_link_5"/>
       <axis xyz="0 1 0"/>
-      <limit effort="5000.0" lower="-3.1416" upper="3.1416" velocity="0.04"/>
+      <limit effort="50000.0" lower="-3.1416" upper="3.1416" velocity="1.0"/>
   </joint>
   <joint name="joint_canadarm2_6" type="revolute">
@@ -213,5 +213,5 @@
       <child link="canadarm2_link_6"/>
       <axis xyz="1 0 0"/>
-      <limit effort="5000.0" lower="-3.1416" upper="3.1416" velocity="0.04"/>
+      <limit effort="50000.0" lower="-3.1416" upper="3.1416" velocity="1.0"/>
   </joint>
   <joint name="joint_canadarm2_7" type="revolute">
@@ -220,5 +220,5 @@
       <child link="canadarm2_link_7"/>
       <axis xyz="0 0 1"/>
-      <limit effort="5000.0" lower="-3.1416" upper="3.1416" velocity="0.04"/>
+      <limit effort="50000.0" lower="-3.1416" upper="3.1416" velocity="1.0"/>
   </joint>
   <xacro:if value="${pt_cameras}">

File: urdf/dextre.urdf.xacro (robot description, xacro)
@@ -112,5 +112,5 @@
       <child link="dextre_body"/>
       <axis xyz="0 0 1"/>
-      <limit effort="1000.0" lower="-3.1416" upper="3.1416" velocity="0.5"/>
+      <limit effort="10000.0" lower="-3.1416" upper="3.1416" velocity="1.0"/>
   </joint>
   <!-- *********************  -->
@@ -246,5 +246,5 @@
       <child link="dextre_arm_1_shoulder_roll"/>
       <axis xyz="1 0 0"/>
-      <limit effort="1000.0" lower="-3.1416" upper="3.1416" velocity="0.5"/>
+      <limit effort="10000.0" lower="-3.1416" upper="3.1416" velocity="1.0"/>
   </joint>
   <!-- joint arm 1 shoulder yaw -->
@@ -254,5 +254,5 @@
       <child link="dextre_arm_1_shoulder_yaw"/>
       <axis xyz="0 0 1"/>
-      <limit effort="1000.0" lower="-3.1416" upper="3.1416" velocity="0.5"/>
+      <limit effort="10000.0" lower="-3.1416" upper="3.1416" velocity="1.0"/>
   </joint>
   <!-- joint arm 1 shoulder pitch -->
@@ -262,5 +262,5 @@
       <child link="dextre_arm_1_shoulder_pitch"/>
       <axis xyz="0 1 0"/>
-      <limit effort="1000.0" lower="-3.1416" upper="3.1416" velocity="0.5"/>
+      <limit effort="10000.0" lower="-3.1416" upper="3.1416" velocity="1.0"/>
   </joint>
   <!-- joint arm 1 elbow pitch -->
@@ -270,5 +270,5 @@
       <child link="dextre_arm_1_elbow_pitch"/>
       <axis xyz="0 1 0"/>
-      <limit effort="1000.0" lower="-3.1416" upper="3.1416" velocity="0.5"/>
+      <limit effort="10000.0" lower="-3.1416" upper="3.1416" velocity="1.0"/>
   </joint>
   <!-- joint arm 1 wrist pitch yaw -->
@@ -278,5 +278,5 @@
       <child link="dextre_arm_1_wrist_pitch_yaw"/>
       <axis xyz="0 1 0"/>
-      <limit effort="1000.0" lower="-3.1416" upper="3.1416" velocity="0.5"/>
+      <limit effort="10000.0" lower="-3.1416" upper="3.1416" velocity="1.0"/>
   </joint>
   <!-- joint arm 1 wrist roll -->
@@ -286,5 +286,5 @@
       <child link="dextre_arm_1_wrist_roll"/>
       <axis xyz="0 0 1"/>
-      <limit effort="1000.0" lower="-3.1416" upper="3.1416" velocity="0.5"/>
+      <limit effort="10000.0" lower="-3.1416" upper="3.1416" velocity="1.0"/>
   </joint>
   <!-- *********************  -->
@@ -420,5 +420,5 @@
       <child link="dextre_arm_2_shoulder_roll"/>
       <axis xyz="1 0 0"/>
-      <limit effort="1000.0" lower="-3.1416" upper="3.1416" velocity="0.5"/>
+      <limit effort="10000.0" lower="-3.1416" upper="3.1416" velocity="1.0"/>
   </joint>
   <!-- joint arm 2 shoulder yaw -->
@@ -428,5 +428,5 @@
       <child link="dextre_arm_2_shoulder_yaw"/>
       <axis xyz="0 0 1"/>
-      <limit effort="1000.0" lower="-3.1416" upper="3.1416" velocity="0.5"/>
+      <limit effort="10000.0" lower="-3.1416" upper="3.1416" velocity="1.0"/>
   </joint>
   <!-- joint arm 2 shoulder pitch -->
@@ -436,5 +436,5 @@
       <child link="dextre_arm_2_shoulder_pitch"/>
       <axis xyz="0 1 0"/>
-      <limit effort="1000.0" lower="-3.1416" upper="3.1416" velocity="0.5"/>
+      <limit effort="10000.0" lower="-3.1416" upper="3.1416" velocity="1.0"/>
   </joint>
   <!-- joint arm 2 elbow pitch -->
@@ -444,5 +444,5 @@
       <child link="dextre_arm_2_elbow_pitch"/>
       <axis xyz="0 1 0"/>
-      <limit effort="1000.0" lower="-3.1416" upper="3.1416" velocity="0.5"/>
+      <limit effort="10000.0" lower="-3.1416" upper="3.1416" velocity="1.0"/>
   </joint>
   <!-- joint arm 2 wrist pitch yaw -->
@@ -452,5 +452,5 @@
       <child link="dextre_arm_2_wrist_pitch_yaw"/>
       <axis xyz="0 1 0"/>
-      <limit effort="1000.0" lower="-3.1416" upper="3.1416" velocity="0.5"/>
+      <limit effort="10000.0" lower="-3.1416" upper="3.1416" velocity="1.0"/>
   </joint>
   <!-- joint arm 2 wrist roll -->
@@ -460,5 +460,5 @@
       <child link="dextre_arm_2_wrist_roll"/>
       <axis xyz="0 0 1"/>
-      <limit effort="1000.0" lower="-3.1416" upper="3.1416" velocity="0.5"/>
+      <limit effort="10000.0" lower="-3.1416" upper="3.1416" velocity="1.0"/>
   </joint>
   <xacro:if value="${pt_cameras}">

File: urdf/mobile_base_system.urdf.xacro (robot description, xacro)
@@ -81,5 +81,5 @@
       <parent link="link_14_s0_truss"/>
       <child link="mobile_base_system"/>
-      <limit effort="1000.0" lower="-15.0" upper="42.0" velocity="0.5"/>
+      <limit effort="100000.0" lower="-15.0" upper="42.0" velocity="5.0"/>
   </joint>
   </xacro:macro>

File: urdf/solar_panels.urdf.xacro (robot description, xacro)
@@ -355,5 +355,5 @@
       <parent link="link_19_p3_truss"/>
       <child link="link_20_p4_truss"/>
-      <limit effort="1000.0" lower="-3.1416" upper="3.1416" velocity="0.5"/>
+      <limit effort="10000.0" lower="-3.1416" upper="3.1416" velocity="1.0"/>
   </joint>
   <!-- Joint to rotate individually panel 1-->
@@ -363,5 +363,5 @@
       <parent link="link_08_p6_truss"/>
       <child link="link_08_p6_truss_01"/>
-      <limit effort="1000.0" lower="-3.1416" upper="3.1416" velocity="0.5"/>
+      <limit effort="10000.0" lower="-3.1416" upper="3.1416" velocity="1.0"/>
   </joint>
   <!-- Joint to rotate individually panel 2 -->
@@ -371,5 +371,5 @@
       <parent link="link_08_p6_truss"/>
       <child link="link_08_p6_truss_02"/>
-      <limit effort="1000.0" lower="-3.1416" upper="3.1416" velocity="0.5"/>
+      <limit effort="10000.0" lower="-3.1416" upper="3.1416" velocity="1.0"/>
   </joint>
   <!-- Joint to rotate individually panel 3 -->
@@ -379,5 +379,5 @@
       <parent link="link_21_p5_truss"/>
       <child link="link_20_p4_truss_01"/>
-      <limit effort="1000.0" lower="-3.1416" upper="3.1416" velocity="0.5"/>
+      <limit effort="10000.0" lower="-3.1416" upper="3.1416" velocity="1.0"/>
   </joint>
   <!-- Joint to rotate individually panel 4 -->
@@ -387,5 +387,5 @@
       <parent link="link_21_p5_truss"/>
       <child link="link_20_p4_truss_02"/>
-      <limit effort="1000.0" lower="-3.1416" upper="3.1416" velocity="0.5"/>
+      <limit effort="10000.0" lower="-3.1416" upper="3.1416" velocity="1.0"/>
   </joint>
   <!-- ************************* -->
@@ -434,5 +434,5 @@
       <parent link="link_22_s3_truss"/>
       <child link="link_23_s4_truss"/>
-      <limit effort="1000.0" lower="-3.1416" upper="3.1416" velocity="0.5"/>
+      <limit effort="10000.0" lower="-3.1416" upper="3.1416" velocity="1.0"/>
   </joint>
   <!-- Joint to rotate individually panel 1-->
@@ -442,5 +442,5 @@
       <parent link="link_24_s5_truss"/>
       <child link="link_23_s4_truss_01"/>
-      <limit effort="1000.0" lower="-3.1416" upper="3.1416" velocity="0.5"/>
+      <limit effort="10000.0" lower="-3.1416" upper="3.1416" velocity="1.0"/>
   </joint>
   <!-- Joint to rotate individually panel 2 -->
@@ -450,5 +450,5 @@
       <parent link="link_24_s5_truss"/>
       <child link="link_23_s4_truss_02"/>
-      <limit effort="1000.0" lower="-3.1416" upper="3.1416" velocity="0.5"/>
+      <limit effort="10000.0" lower="-3.1416" upper="3.1416" velocity="1.0"/>
   </joint>
   <!-- Joint to rotate individually panel 3 -->
@@ -458,5 +458,5 @@
       <parent link="link_32_s6_truss"/>
       <child link="link_32_s6_truss_01"/>
-      <limit effort="1000.0" lower="-3.1416" upper="3.1416" velocity="0.5"/>
+      <limit effort="10000.0" lower="-3.1416" upper="3.1416" velocity="1.0"/>
   </joint>
   <!-- Joint to rotate individually panel 4 -->
@@ -466,5 +466,5 @@
       <parent link="link_32_s6_truss"/>
       <child link="link_32_s6_truss_02"/>
-      <limit effort="1000.0" lower="-3.1416" upper="3.1416" velocity="0.5"/>
+      <limit effort="10000.0" lower="-3.1416" upper="3.1416" velocity="1.0"/>
   </joint>
   </xacro:macro>
