Commit message: Added dextre 7th DOF

File: urdf/dextre.gazebo.xacro (robot description, xacro)
@@ -33,5 +33,11 @@
           <state_interface name="effort"/>
       </joint>
-      <joint name="joint_dextre_arm_1_wrist_pitch_yaw">
+      <joint name="joint_dextre_arm_1_wrist_pitch">
+          <command_interface name="${command_interface}"/>
+          <state_interface name="position"/>
+          <state_interface name="velocity"/>
+          <state_interface name="effort"/>
+      </joint>
+      <joint name="joint_dextre_arm_1_wrist_yaw">
           <command_interface name="${command_interface}"/>
           <state_interface name="position"/>
@@ -70,5 +76,11 @@
           <state_interface name="effort"/>
       </joint>
-      <joint name="joint_dextre_arm_2_wrist_pitch_yaw">
+      <joint name="joint_dextre_arm_2_wrist_pitch">
+          <command_interface name="${command_interface}"/>
+          <state_interface name="position"/>
+          <state_interface name="velocity"/>
+          <state_interface name="effort"/>
+      </joint>
+      <joint name="joint_dextre_arm_2_wrist_yaw">
           <command_interface name="${command_interface}"/>
           <state_interface name="position"/>

File: urdf/dextre.urdf.xacro (robot description, xacro)
@@ -197,21 +197,41 @@
    </collision>
   </link>
-  <!-- ******* Link Arm 1 Wrist Pitch Yaw *******  -->
-  <link name="dextre_arm_1_wrist_pitch_yaw">
-   <inertial>
-     <origin xyz="0 0 0.0" rpy="0 0 0"/>
-     <mass value="1"/>
-     <inertia ixx="100"  ixy="0"  ixz="0" iyy="100" iyz="0" izz="100" />
-   </inertial>
-   <visual>
-     <origin xyz="0 0 0" rpy="0 0 0" />
-     <geometry>
-       <mesh filename="package://iss_description/meshes/dextre/arm_1/wrist_pitch_yaw.dae" scale="1 1 1"/>
-     </geometry>
-   </visual>
-   <collision>
-     <origin xyz="0 0 0" rpy="0 0 0"/>
-     <geometry>
-       <mesh filename="package://iss_description/meshes/dextre/arm_1/wrist_pitch_yaw.dae" scale="1 1 1"/>
+  <!-- ******* Link Arm 1 Wrist Pitch *******  -->
+  <link name="dextre_arm_1_wrist_pitch">
+   <inertial>
+     <origin xyz="0 0 0.0" rpy="0 0 0"/>
+     <mass value="1"/>
+     <inertia ixx="100"  ixy="0"  ixz="0" iyy="100" iyz="0" izz="100" />
+   </inertial>
+   <visual>
+     <origin xyz="0 0 0" rpy="0 0 0" />
+     <geometry>
+       <mesh filename="package://iss_description/meshes/dextre/arm_1/wrist_pitch.dae" scale="1 1 1"/>
+     </geometry>
+   </visual>
+   <collision>
+     <origin xyz="0 0 0" rpy="0 0 0"/>
+     <geometry>
+       <mesh filename="package://iss_description/meshes/dextre/arm_1/wrist_pitch.dae" scale="1 1 1"/>
+     </geometry>
+   </collision>
+  </link>
+  <!-- ******* Link Arm 1 Wrist Yaw *******  -->
+  <link name="dextre_arm_1_wrist_yaw">
+   <inertial>
+     <origin xyz="0 0.0 0.0" rpy="0 0 0"/>
+     <mass value="1"/>
+     <inertia ixx="100"  ixy="0"  ixz="0" iyy="100" iyz="0" izz="100" />
+   </inertial>
+   <visual>
+     <origin xyz="0 -0.11 0" rpy="0 0 0" />
+     <geometry>
+       <mesh filename="package://iss_description/meshes/dextre/arm_1/wrist_yaw.dae" scale="1 1 1"/>
+     </geometry>
+   </visual>
+   <collision>
+     <origin xyz="0 -0.11 0" rpy="0 0 0"/>
+     <geometry>
+       <mesh filename="package://iss_description/meshes/dextre/arm_1/wrist_yaw.dae" scale="1 1 1"/>
      </geometry>
    </collision>
@@ -272,10 +292,18 @@
       <limit effort="10000.0" lower="-3.1416" upper="3.1416" velocity="1.0"/>
   </joint>
-  <!-- joint arm 1 wrist pitch yaw -->
-  <joint name="joint_dextre_arm_1_wrist_pitch_yaw" type="revolute">
+  <!-- joint arm 1 wrist pitch -->
+  <joint name="joint_dextre_arm_1_wrist_pitch" type="revolute">
       <origin rpy="0 0 0" xyz="-1.0873 0.3271 -0.012581"/>
       <parent link="dextre_arm_1_elbow_pitch"/>
-      <child link="dextre_arm_1_wrist_pitch_yaw"/>
+      <child link="dextre_arm_1_wrist_pitch"/>
       <axis xyz="0 1 0"/>
+      <limit effort="10000.0" lower="-3.1416" upper="3.1416" velocity="1.0"/>
+  </joint>
+  <!-- joint arm 1 wrist yaw -->
+  <joint name="joint_dextre_arm_1_wrist_yaw" type="revolute">
+      <origin rpy="0 0 0" xyz="-0.01 0.11 0.0"/>
+      <parent link="dextre_arm_1_wrist_pitch"/>
+      <child link="dextre_arm_1_wrist_yaw"/>
+      <axis xyz="1 0 0"/>
       <limit effort="10000.0" lower="-3.1416" upper="3.1416" velocity="1.0"/>
   </joint>
@@ -283,5 +311,5 @@
   <joint name="joint_dextre_arm_1_wrist_roll" type="revolute">
       <origin rpy="0 0 0" xyz="-0.28177 0.11183 -0.12003"/>
-      <parent link="dextre_arm_1_wrist_pitch_yaw"/>
+      <parent link="dextre_arm_1_wrist_yaw"/>
       <child link="dextre_arm_1_wrist_roll"/>
       <axis xyz="0 0 1"/>
@@ -371,21 +399,41 @@
    </collision>
   </link>
-  <!-- ******* Link Arm 2 Wrist Pitch Yaw *******  -->
-  <link name="dextre_arm_2_wrist_pitch_yaw">
-   <inertial>
-     <origin xyz="0 0 0.0" rpy="0 0 0"/>
-     <mass value="1"/>
-     <inertia ixx="100"  ixy="0"  ixz="0" iyy="100" iyz="0" izz="100" />
-   </inertial>
-   <visual>
-     <origin xyz="0 0 0" rpy="0 0 0" />
-     <geometry>
-       <mesh filename="package://iss_description/meshes/dextre/arm_2/wrist_pitch_yaw.dae" scale="1 1 1"/>
-     </geometry>
-   </visual>
-   <collision>
-     <origin xyz="0 0 0" rpy="0 0 0"/>
-     <geometry>
-       <mesh filename="package://iss_description/meshes/dextre/arm_2/wrist_pitch_yaw.dae" scale="1 1 1"/>
+  <!-- ******* Link Arm 2 Wrist Pitch *******  -->
+  <link name="dextre_arm_2_wrist_pitch">
+   <inertial>
+     <origin xyz="0 0 0.0" rpy="0 0 0"/>
+     <mass value="1"/>
+     <inertia ixx="100"  ixy="0"  ixz="0" iyy="100" iyz="0" izz="100" />
+   </inertial>
+   <visual>
+     <origin xyz="0 0 0" rpy="0 0 0" />
+     <geometry>
+       <mesh filename="package://iss_description/meshes/dextre/arm_2/wrist_pitch.dae" scale="1 1 1"/>
+     </geometry>
+   </visual>
+   <collision>
+     <origin xyz="0 0 0" rpy="0 0 0"/>
+     <geometry>
+       <mesh filename="package://iss_description/meshes/dextre/arm_2/wrist_pitch.dae" scale="1 1 1"/>
+     </geometry>
+   </collision>
+  </link>
+  <!-- ******* Link Arm 2 Wrist Yaw *******  -->
+  <link name="dextre_arm_2_wrist_yaw">
+   <inertial>
+     <origin xyz="0.0 0 0.0" rpy="0 0 0"/>
+     <mass value="1"/>
+     <inertia ixx="100"  ixy="0"  ixz="0" iyy="100" iyz="0" izz="100" />
+   </inertial>
+   <visual>
+     <origin xyz="0 -0.11 0" rpy="0 0 0" />
+     <geometry>
+       <mesh filename="package://iss_description/meshes/dextre/arm_2/wrist_yaw.dae" scale="1 1 1"/>
+     </geometry>
+   </visual>
+   <collision>
+     <origin xyz="0 -0.11 0" rpy="0 0 0"/>
+     <geometry>
+       <mesh filename="package://iss_description/meshes/dextre/arm_2/wrist_yaw.dae" scale="1 1 1"/>
      </geometry>
    </collision>
@@ -447,9 +495,17 @@
   </joint>
   <!-- joint arm 2 wrist pitch yaw -->
-  <joint name="joint_dextre_arm_2_wrist_pitch_yaw" type="revolute">
+  <joint name="joint_dextre_arm_2_wrist_pitch" type="revolute">
       <origin rpy="0 0 0" xyz="1.0873 0.3271 -0.012577"/>
       <parent link="dextre_arm_2_elbow_pitch"/>
-      <child link="dextre_arm_2_wrist_pitch_yaw"/>
+      <child link="dextre_arm_2_wrist_pitch"/>
       <axis xyz="0 1 0"/>
+      <limit effort="10000.0" lower="-3.1416" upper="3.1416" velocity="1.0"/>
+  </joint>
+  <!-- joint arm 2 wrist yaw -->
+  <joint name="joint_dextre_arm_2_wrist_yaw" type="revolute">
+      <origin rpy="0 0 0" xyz="0.01 0.11 0.0"/>
+      <parent link="dextre_arm_2_wrist_pitch"/>
+      <child link="dextre_arm_2_wrist_yaw"/>
+      <axis xyz="1 0 0"/>
       <limit effort="10000.0" lower="-3.1416" upper="3.1416" velocity="1.0"/>
   </joint>
@@ -457,5 +513,5 @@
   <joint name="joint_dextre_arm_2_wrist_roll" type="revolute">
       <origin rpy="0 0 0" xyz="0.28178 0.11183 -0.12001"/>
-      <parent link="dextre_arm_2_wrist_pitch_yaw"/>
+      <parent link="dextre_arm_2_wrist_yaw"/>
       <child link="dextre_arm_2_wrist_roll"/>
       <axis xyz="0 0 1"/>

File: urdf/mobile_base_system.gazebo.xacro (robot description, xacro)
@@ -4,5 +4,7 @@
       <joint name="joint_mbs">
           <command_interface name="${command_interface}"/>
-          <state_interface name="position"/>
+          <state_interface name="position">
+            <param name="initial_value">-13.0</param>
+          </state_interface>
           <state_interface name="velocity"/>
           <state_interface name="effort"/>

File: urdf/mobile_servicing_system.gazebo.xacro (robot description, xacro)
@@ -29,4 +29,14 @@
       </xacro:if>
     </ros2_control>
+    <!-- Plugin to attach/detach objects to Dextre arm 1 -->
+    <gazebo>
+      <plugin filename="libDynamicDetachableJoint.so"
+              name="gz::sim::systems::DynamicDetachableJoint">
+        <parent_link>dextre_arm_1_wrist_roll</parent_link>
+        <service_name>/payload/attach_detach</service_name>
+        <output_topic>/payload/child_state</output_topic>
+        <attach_distance>10.0</attach_distance> <!-- 10 cm -->
+      </plugin>
+    </gazebo>
   <gazebo>
       <plugin filename="gz_ros2_control-system" name="gz_ros2_control::GazeboSimROS2ControlPlugin">

File: urdf/solar_panels.gazebo.xacro (robot description, xacro)
@@ -44,5 +44,7 @@
       <joint name="joint_starboard_bga_1">
           <command_interface name="${command_interface}"/>
-          <state_interface name="position"/>
+          <state_interface name="position">
+            <param name="initial_value">1.5708</param>
+          </state_interface>
           <state_interface name="velocity"/>
           <state_interface name="effort"/>
