Commit message: Added dextre DOF

File: urdf/dextre.urdf.xacro (robot description, xacro)
@@ -313,4 +313,12 @@
       <parent link="dextre_arm_1_wrist_yaw"/>
       <child link="dextre_arm_1_wrist_roll"/>
+      <axis xyz="0 0 1"/>
+      <limit effort="10000.0" lower="-3.1416" upper="3.1416" velocity="1.0"/>
+  </joint>
+  <link name="dextre_arm_1_ee_ref"/>
+  <joint name="joint_dextre_arm_1_ee_ref" type="fixed">
+      <origin rpy="-1.5708 0.0 1.5708" xyz="0.0 0.0 -1.0"/>
+      <parent link="dextre_arm_1_wrist_roll"/>
+      <child link="dextre_arm_1_ee_ref"/>
       <axis xyz="0 0 1"/>
       <limit effort="10000.0" lower="-3.1416" upper="3.1416" velocity="1.0"/>
