Commit message: Adds pan tilt cameras to sim model, creates bridges for cameras, updates candarm2 model to have more realistic physics properties, adds positionable sun in world with script to change zenith angle, ensure sim time used in gz contollers, updates move example to use action servers, and adds test example launch arg (default false)

File: robots/mobile_servicing_system.urdf.xacro (robot description, xacro)
@@ -5,4 +5,5 @@
   <xacro:include filename="$(find iss_description)/urdf/dextre.urdf.xacro"/>
   <xacro:include filename="$(find iss_description)/urdf/solar_panels.urdf.xacro"/>
+  <xacro:include filename="$(find iss_description)/urdf/etvcg_cameras.urdf.xacro"/>
   <!-- Gazebo -->
   <xacro:include filename="$(find iss_description)/urdf/mobile_servicing_system.gazebo.xacro"/>
@@ -16,3 +17,5 @@
   <xacro:dextre parent="canadarm2_link_7"/>
   <xacro:canadarm2 parent="mobile_base_system"/>
+  <!-- ETV-CG Cameras -->
+  <xacro:etvcg_cameras parent="root"/>
 </robot>

File: urdf/canadarm2.urdf.xacro (robot description, xacro)
@@ -1,5 +1,6 @@
 <?xml version="1.0"?>
 <robot name="canadarm2" xmlns:xacro="http://www.ros.org/wiki/xacro">
-  <!-- CANADARM2 -->
+  <xacro:include filename="$(find iss_description)/urdf/pt_camera.urdf.xacro"/>
+  <xacro:include filename="$(find iss_description)/urdf/pt_camera.gazebo.xacro"/>
   <xacro:macro name="canadarm2" params=" parent:='' ">
   <link name="pdgf"/>
@@ -10,10 +11,9 @@
       <child link="pdgf_forward"/>
   </joint>
-  <!-- ******* Link Base *******  -->
   <link name="canadarm2_base">
    <inertial>
      <origin xyz="0 0 0.0" rpy="0 0 0"/>
-     <mass value="1"/>
-     <inertia ixx="100"  ixy="0"  ixz="0" iyy="100" iyz="0" izz="100" />
+     <mass value="200.0"/>
+     <inertia ixx="10.0"  ixy="0"  ixz="0" iyy="10.0" iyz="0" izz="10.0" />
    </inertial>
    <visual>
@@ -30,130 +30,123 @@
    </collision>
   </link>
-  <!-- ******* Link 1 *******  -->
   <link name="canadarm2_link_1">
     <inertial>
+      <origin xyz="0 -0.5 0.0" rpy="0 0 0"/>
+      <mass value="140.0"/>
+      <inertia ixx="8.0"  ixy="0"  ixz="0" iyy="5.0" iyz="0" izz="8.0" />
+    </inertial>
+    <visual>
+      <origin xyz="0 0 0" rpy="0.0 -0.488692 0.663225" />
+      <geometry>
+        <mesh filename="package://iss_description/meshes/canadarm2/link_1.dae" scale="1 1 1"/>
+      </geometry>
+    </visual>
+    <collision>
+      <origin xyz="0 0 0" rpy="0.0 -0.488692 0.663225"/>
+      <geometry>
+        <mesh filename="package://iss_description/meshes/canadarm2/link_1.dae" scale="1 1 1"/>
+      </geometry>
+    </collision>
+   </link>
+  <link name="canadarm2_link_2">
+    <inertial>
       <origin xyz="0 0 0.0" rpy="0 0 0"/>
-      <mass value="1"/>
-      <inertia ixx="100"  ixy="0"  ixz="0" iyy="100" iyz="0" izz="100" />
-    </inertial>
-    <visual>
-      <origin xyz="0 0 0" rpy="0.0 -0.488692 0.663225" /> <!-- Blender: 0 -28 38-->
-      <geometry>
-        <mesh filename="package://iss_description/meshes/canadarm2/link_1.dae" scale="1 1 1"/>
-      </geometry>
-    </visual>
-    <collision>
-      <origin xyz="0 0 0" rpy="0.0 -0.488692 0.663225"/>
-      <geometry>
-        <mesh filename="package://iss_description/meshes/canadarm2/link_1.dae" scale="1 1 1"/>
-      </geometry>
-    </collision>
-   </link>
-  <!-- ******* Link 2 *******  -->
-  <link name="canadarm2_link_2">
+      <mass value="120.0"/>
+      <inertia ixx="8.0"  ixy="0"  ixz="0" iyy="8.0" iyz="0" izz="5.0" />
+    </inertial>
+    <visual>
+      <origin xyz="0 0 0" rpy="0 -0.49131018 0" />
+      <geometry>
+        <mesh filename="package://iss_description/meshes/canadarm2/link_2.dae" scale="1 1 1"/>
+      </geometry>
+    </visual>
+    <collision>
+      <origin xyz="0 0 0" rpy="0 -0.49131018 0"/>
+      <geometry>
+        <mesh filename="package://iss_description/meshes/canadarm2/link_2.dae" scale="1 1 1"/>
+      </geometry>
+    </collision>
+   </link>
+  <link name="canadarm2_link_3">
+    <inertial>
+      <origin xyz="-3.0 0 0.0" rpy="0 0 0"/>
+      <mass value="100.0"/>
+      <inertia ixx="5.0"  ixy="0"  ixz="0" iyy="200.0" iyz="0" izz="200.0" />
+    </inertial>
+    <visual>
+      <origin xyz="0 0 0" rpy="0 0 0" />
+      <geometry>
+        <mesh filename="package://iss_description/meshes/canadarm2/link_3.dae" scale="1 1 1"/>
+      </geometry>
+    </visual>
+    <collision>
+      <origin xyz="0 0 0" rpy="0 0 0"/>
+      <geometry>
+        <mesh filename="package://iss_description/meshes/canadarm2/link_3.dae" scale="1 1 1"/>
+      </geometry>
+    </collision>
+   </link>
+  <link name="canadarm2_link_4">
+    <inertial>
+      <origin xyz="0 -3.5 0.0" rpy="0 0 0"/>
+      <mass value="150.0"/>
+      <inertia ixx="615.0"  ixy="0"  ixz="0" iyy="5.0" iyz="0" izz="615.0" />
+    </inertial>
+    <visual>
+      <origin xyz="0 0 0" rpy="0 0 0" />
+      <geometry>
+        <mesh filename="package://iss_description/meshes/canadarm2/link_4.dae" scale="1 1 1"/>
+      </geometry>
+    </visual>
+    <collision>
+      <origin xyz="0 0 0" rpy="0 0 0"/>
+      <geometry>
+        <mesh filename="package://iss_description/meshes/canadarm2/link_4.dae" scale="1 1 1"/>
+      </geometry>
+    </collision>
+   </link>
+  <link name="canadarm2_link_5">
+    <inertial>
+      <origin xyz="0 0 3.5" rpy="0 0 0"/>
+      <mass value="150.0"/>
+      <inertia ixx="615.0"  ixy="0"  ixz="0" iyy="615.0" iyz="0" izz="5.0" />
+    </inertial>
+    <visual>
+      <origin xyz="0 0 0" rpy="0 0 0" />
+      <geometry>
+        <mesh filename="package://iss_description/meshes/canadarm2/link_5.dae" scale="1 1 1"/>
+      </geometry>
+    </visual>
+    <collision>
+      <origin xyz="0 0 0" rpy="0 0 0"/>
+      <geometry>
+        <mesh filename="package://iss_description/meshes/canadarm2/link_5.dae" scale="1 1 1"/>
+      </geometry>
+    </collision>
+   </link>
+  <link name="canadarm2_link_6">
     <inertial>
       <origin xyz="0 0 0.0" rpy="0 0 0"/>
-      <mass value="1"/>
-      <inertia ixx="100"  ixy="0"  ixz="0" iyy="100" iyz="0" izz="100" />
-    </inertial>
-    <visual>
-      <origin xyz="0 0 0" rpy="0 -0.49131018 0" /> <!-- Blender: 0.0 -28.15 0.0-->
-      <geometry>
-        <mesh filename="package://iss_description/meshes/canadarm2/link_2.dae" scale="1 1 1"/>
-      </geometry>
-    </visual>
-    <collision>
-      <origin xyz="0 0 0" rpy="0 -0.49131018 0"/>
-      <geometry>
-        <mesh filename="package://iss_description/meshes/canadarm2/link_2.dae" scale="1 1 1"/>
-      </geometry>
-    </collision>
-   </link>
-  <!-- ******* Link 3 *******  -->
-  <link name="canadarm2_link_3">
+      <mass value="120.0"/>
+      <inertia ixx="8.0"  ixy="0"  ixz="0" iyy="8.0" iyz="0" izz="5.0" />
+    </inertial>
+    <visual>
+      <origin xyz="0 0 0" rpy="0 0 0" />
+      <geometry>
+        <mesh filename="package://iss_description/meshes/canadarm2/link_6.dae" scale="1 1 1"/>
+      </geometry>
+    </visual>
+    <collision>
+      <origin xyz="0 0 0" rpy="0 0 0"/>
+      <geometry>
+        <mesh filename="package://iss_description/meshes/canadarm2/link_6.dae" scale="1 1 1"/>
+      </geometry>
+    </collision>
+   </link>
+  <link name="canadarm2_link_7">
     <inertial>
       <origin xyz="0 0 0.0" rpy="0 0 0"/>
-      <mass value="1"/>
-      <inertia ixx="100"  ixy="0"  ixz="0" iyy="100" iyz="0" izz="100" />
-    </inertial>
-    <visual>
-      <origin xyz="0 0 0" rpy="0 0 0" />
-      <geometry>
-        <mesh filename="package://iss_description/meshes/canadarm2/link_3.dae" scale="1 1 1"/>
-      </geometry>
-    </visual>
-    <collision>
-      <origin xyz="0 0 0" rpy="0 0 0"/>
-      <geometry>
-        <mesh filename="package://iss_description/meshes/canadarm2/link_3.dae" scale="1 1 1"/>
-      </geometry>
-    </collision>
-   </link>
-  <!-- ******* Link 4 *******  -->
-  <link name="canadarm2_link_4">
-    <inertial>
-      <origin xyz="0 0 0.0" rpy="0 0 0"/>
-      <mass value="1"/>
-      <inertia ixx="100"  ixy="0"  ixz="0" iyy="100" iyz="0" izz="100" />
-    </inertial>
-    <visual>
-      <origin xyz="0 0 0" rpy="0 0 0" />
-      <geometry>
-        <mesh filename="package://iss_description/meshes/canadarm2/link_4.dae" scale="1 1 1"/>
-      </geometry>
-    </visual>
-    <collision>
-      <origin xyz="0 0 0" rpy="0 0 0"/>
-      <geometry>
-        <mesh filename="package://iss_description/meshes/canadarm2/link_4.dae" scale="1 1 1"/>
-      </geometry>
-    </collision>
-   </link>
-  <!-- ******* Link 5 *******  -->
-  <link name="canadarm2_link_5">
-    <inertial>
-      <origin xyz="0 0 0.0" rpy="0 0 0"/>
-      <mass value="1"/>
-      <inertia ixx="100"  ixy="0"  ixz="0" iyy="100" iyz="0" izz="100" />
-    </inertial>
-    <visual>
-      <origin xyz="0 0 0" rpy="0 0 0" />
-      <geometry>
-        <mesh filename="package://iss_description/meshes/canadarm2/link_5.dae" scale="1 1 1"/>
-      </geometry>
-    </visual>
-    <collision>
-      <origin xyz="0 0 0" rpy="0 0 0"/>
-      <geometry>
-        <mesh filename="package://iss_description/meshes/canadarm2/link_5.dae" scale="1 1 1"/>
-      </geometry>
-    </collision>
-   </link>
-  <!-- ******* Link 6 *******  -->
-  <link name="canadarm2_link_6">
-    <inertial>
-      <origin xyz="0 0 0.0" rpy="0 0 0"/>
-      <mass value="1"/>
-      <inertia ixx="100"  ixy="0"  ixz="0" iyy="100" iyz="0" izz="100" />
-    </inertial>
-    <visual>
-      <origin xyz="0 0 0" rpy="0 0 0" />
-      <geometry>
-        <mesh filename="package://iss_description/meshes/canadarm2/link_6.dae" scale="1 1 1"/>
-      </geometry>
-    </visual>
-    <collision>
-      <origin xyz="0 0 0" rpy="0 0 0"/>
-      <geometry>
-        <mesh filename="package://iss_description/meshes/canadarm2/link_6.dae" scale="1 1 1"/>
-      </geometry>
-    </collision>
-   </link>
-  <!-- ******* Link 7 *******  -->
-  <link name="canadarm2_link_7">
-    <inertial>
-      <origin xyz="0 0 0.0" rpy="0 0 0"/>
-      <mass value="1"/>
-      <inertia ixx="100"  ixy="0"  ixz="0" iyy="100" iyz="0" izz="100" />
+      <mass value="200.0"/>
+      <inertia ixx="10.0"  ixy="0"  ixz="0" iyy="10.0" iyz="0" izz="10.0" />
     </inertial>
     <visual>
@@ -180,13 +173,11 @@
       <child link="canadarm2_base"/>
   </joint>
-  <!-- joint 1 -->
   <joint name="joint_canadarm2_1" type="revolute">
-      <origin rpy="0 0 0" xyz="0.0 -1.2388 0.0"/> <!-- -0.66927 -0.97994 0.3556 -->
+      <origin rpy="0 0 0" xyz="0.0 -1.2388 0.0"/>
       <parent link="canadarm2_base"/>
       <child link="canadarm2_link_1"/>
       <axis xyz="0 1 0"/>
-      <limit effort="1000.0" lower="-3.1416" upper="3.1416" velocity="0.5"/>
-  </joint>
-  <!-- joint 2 -->
+      <limit effort="10000.0" lower="-3.1416" upper="3.1416" velocity="0.04"/>
+  </joint>
   <joint name="joint_canadarm2_2" type="revolute">
       <origin rpy="0 0 0" xyz="-0.005874 -0.22963 0.35801"/>
@@ -194,7 +185,6 @@
       <child link="canadarm2_link_2"/>
       <axis xyz="0 0 1"/>
-      <limit effort="1000.0" lower="-3.1416" upper="3.1416" velocity="0.5"/>
-  </joint>
-  <!-- joint 3 -->
+      <limit effort="10000.0" lower="-3.1416" upper="3.1416" velocity="0.04"/>
+  </joint>
   <joint name="joint_canadarm2_3" type="revolute">
       <origin rpy="0 0 0" xyz="0.13387 -0.31415 0.25363"/>
@@ -202,7 +192,6 @@
       <child link="canadarm2_link_3"/>
       <axis xyz="0 1 0"/>
-      <limit effort="1000.0" lower="-3.1416" upper="3.1416" velocity="0.5"/>
-  </joint>
-  <!-- joint 4 -->
+      <limit effort="10000.0" lower="-3.1416" upper="3.1416" velocity="0.04"/>
+  </joint>
   <joint name="joint_canadarm2_4" type="revolute">
       <origin rpy="0 0 0" xyz="-7.3435 -0.57517 0.004392"/>
@@ -210,7 +199,6 @@
       <child link="canadarm2_link_4"/>
       <axis xyz="0 1 0"/>
-      <limit effort="1000.0" lower="-3.1416" upper="3.1416" velocity="0.5"/>
-  </joint>
-  <!-- joint 5 -->
+      <limit effort="10000.0" lower="-3.1416" upper="3.1416" velocity="0.04"/>
+  </joint>
   <joint name="joint_canadarm2_5" type="revolute">
       <origin rpy="0 0 0" xyz="0.004395 -0.57517 7.3435"/>
@@ -218,7 +206,6 @@
       <child link="canadarm2_link_5"/>
       <axis xyz="0 1 0"/>
-      <limit effort="1000.0" lower="-3.1416" upper="3.1416" velocity="0.5"/>
-  </joint>
-  <!-- joint 6 -->
+      <limit effort="5000.0" lower="-3.1416" upper="3.1416" velocity="0.04"/>
+  </joint>
   <joint name="joint_canadarm2_6" type="revolute">
       <origin rpy="0 0 0" xyz="-0.28758 -0.3134 0.002192"/>
@@ -226,7 +213,6 @@
       <child link="canadarm2_link_6"/>
       <axis xyz="1 0 0"/>
-      <limit effort="1000.0" lower="-3.1416" upper="3.1416" velocity="0.5"/>
-  </joint>
-  <!-- joint 7 -->
+      <limit effort="5000.0" lower="-3.1416" upper="3.1416" velocity="0.04"/>
+  </joint>
   <joint name="joint_canadarm2_7" type="revolute">
       <origin rpy="0 0 0" xyz="-0.31341 -0.002199 0.28759"/>
@@ -234,6 +220,28 @@
       <child link="canadarm2_link_7"/>
       <axis xyz="0 0 1"/>
-      <limit effort="1000.0" lower="-3.1416" upper="3.1416" velocity="0.5"/>
-  </joint>
+      <limit effort="5000.0" lower="-3.1416" upper="3.1416" velocity="0.04"/>
+  </joint>
+  <xacro:pt_camera prefix="boom_a_clpa" parent_link="canadarm2_link_3">
+    <origin xyz="-4.591 0.259 0.0" rpy="1.5708 0.0 1.5708"/>
+  </xacro:pt_camera>
+  <xacro:pt_camera_gazebo
+    prefix="boom_a_clpa"
+    image_width="1024"
+    image_height="1024"
+    horizontal_fov="0.896"
+    update_rate="30.0"
+    enable_lens_flare="true"
+    lens_flare_scale="5.0"/>
+  <xacro:pt_camera prefix="boom_b_clpa" parent_link="canadarm2_link_4">
+    <origin xyz="0.142 -0.847 2.735" rpy="0.0 0.0 0.0"/>
+  </xacro:pt_camera>
+  <xacro:pt_camera_gazebo
+    prefix="boom_b_clpa"
+    image_width="1024"
+    image_height="1024"
+    horizontal_fov="0.896"
+    update_rate="30.0"
+    enable_lens_flare="true"
+    lens_flare_scale="5.0"/>
  </xacro:macro>
 </robot>

File: urdf/dextre.urdf.xacro (robot description, xacro)
@@ -1,4 +1,6 @@
 <?xml version="1.0"?>
 <robot name="dextre" xmlns:xacro="http://www.ros.org/wiki/xacro">
+  <xacro:include filename="$(find iss_description)/urdf/pt_camera.urdf.xacro"/>
+  <xacro:include filename="$(find iss_description)/urdf/pt_camera.gazebo.xacro"/>
   <!-- DEXTRE -->
   <xacro:macro name="dextre" params=" parent:='' ">
@@ -460,4 +462,28 @@
       <limit effort="1000.0" lower="-3.1416" upper="3.1416" velocity="0.5"/>
   </joint>
+  <!-- Outrigger 1 CLPA Camera on tool_platform -->
+  <xacro:pt_camera prefix="outrigger_1_clpa" parent_link="dextre_tool_platform">
+    <origin xyz="1.368 0.300 0.314" rpy="1.5708 0.0 0.0"/>
+  </xacro:pt_camera>
+  <xacro:pt_camera_gazebo
+    prefix="outrigger_1_clpa"
+    image_width="1024"
+    image_height="1024"
+    horizontal_fov="0.896"
+    update_rate="30.0"
+    enable_lens_flare="true"
+    lens_flare_scale="5.0"/>
+  <!-- Outrigger 2 CLPA Camera on tool_platform -->
+  <xacro:pt_camera prefix="outrigger_2_clpa" parent_link="dextre_tool_platform">
+    <origin xyz="-1.368 0.300 0.314" rpy="1.5708 0.0 0.0"/>
+  </xacro:pt_camera>
+  <xacro:pt_camera_gazebo
+    prefix="outrigger_2_clpa"
+    image_width="1024"
+    image_height="1024"
+    horizontal_fov="0.896"
+    update_rate="30.0"
+    enable_lens_flare="true"
+    lens_flare_scale="5.0"/>
   </xacro:macro>
 </robot>

File: urdf/mobile_servicing_system.gazebo.xacro (robot description, xacro)
@@ -5,4 +5,5 @@
   <xacro:include filename="$(find iss_description)/urdf/dextre.gazebo.xacro"/>
   <xacro:include filename="$(find iss_description)/urdf/solar_panels.gazebo.xacro"/>
+  <xacro:include filename="$(find iss_description)/urdf/pt_camera.gazebo.xacro"/>
   <xacro:macro name="mobile_servicing_system_gazebo" params="command_interface:=position">
     <ros2_control name="GazeboSystem" type="system">
@@ -14,4 +15,13 @@
       <xacro:dextre_ros2_control_joints command_interface="${command_interface}"/>
       <xacro:solar_panels_ros2_control_joints command_interface="${command_interface}"/>
+      <!-- Pan-Tilt Camera Joints -->
+      <xacro:pt_camera_ros2_control prefix="boom_a_clpa"/>
+      <xacro:pt_camera_ros2_control prefix="boom_b_clpa"/>
+      <xacro:pt_camera_ros2_control prefix="outrigger_1_clpa"/>
+      <xacro:pt_camera_ros2_control prefix="outrigger_2_clpa"/>
+      <xacro:pt_camera_ros2_control prefix="etvcg_cp3"/>
+      <xacro:pt_camera_ros2_control prefix="etvcg_cp8"/>
+      <xacro:pt_camera_ros2_control prefix="etvcg_cp9"/>
+      <xacro:pt_camera_ros2_control prefix="etvcg_cp13"/>
     </ros2_control>
   <gazebo>
@@ -24,36 +34,4 @@
       </plugin>
   </gazebo>
-  <!-- Simulate camera at the end of big arm-->
-  <link name="dextre_arm_2_dummy_camera_link"/>
-  <joint name="dextre_2_camera_joint" type="fixed">
-    <parent link="dextre_arm_2_wrist_roll"/>
-    <child link="dextre_arm_2_dummy_camera_link"/>
-    <origin xyz="0 0 -0.96" rpy="0.0 0.0 0.0"/>
-  </joint>
-  <gazebo reference="dextre_arm_2_dummy_camera_link">
-      <sensor type="camera" name="camera_sensor">
-          <visualize>1</visualize>
-          <update_rate>10.0</update_rate>
-          <camera>
-              <pose>1.0 0 0 0 0 -1.57</pose>
-              <horizontal_fov>1.3962634</horizontal_fov>
-              <image>
-                  <width>800</width>
-                  <height>800</height>
-                  <format>R8G8B8</format>
-              </image>
-              <clip>
-              <near>0.01</near>
-              <far>100</far>
-              </clip>
-              <noise>
-              <type>gaussian</type>
-              <stddev>0.007</stddev>
-              </noise>
-          </camera>
-          <always_on>1</always_on>
-          <topic>image_raw</topic>
-      </sensor>
-  </gazebo>
   </xacro:macro>
 </robot>
