Commit message: Added if simulate cameras to opt to simulate them or not

File: robots/mobile_servicing_system.urdf.xacro (robot description, xacro)
@@ -6,7 +6,9 @@
   <xacro:include filename="$(find iss_description)/urdf/solar_panels.urdf.xacro"/>
   <xacro:include filename="$(find iss_description)/urdf/etvcg_cameras.urdf.xacro"/>
+  <xacro:arg name="etv_cg_cameras" default="True" />
+  <xacro:arg name="pt_cameras" default="True" />
   <!-- Gazebo -->
   <xacro:include filename="$(find iss_description)/urdf/mobile_servicing_system.gazebo.xacro"/>
-  <xacro:mobile_servicing_system_gazebo command_interface="position"/>
+  <xacro:mobile_servicing_system_gazebo command_interface="position" etv_cg_cameras="$(arg etv_cg_cameras)" pt_cameras="$(arg pt_cameras)"/>
   <!-- ISS and Mobile Base System -->
   <link name="world"/>
@@ -15,7 +17,9 @@
   <xacro:solar_panels parent="link_14_s0_truss"/>
   <!-- Canadarm2 and Dextre -->
-  <xacro:dextre parent="canadarm2_link_7"/>
-  <xacro:canadarm2 parent="mobile_base_system"/>
+  <xacro:dextre parent="canadarm2_link_7" pt_cameras="$(arg pt_cameras)"/>
+  <xacro:canadarm2 parent="mobile_base_system" pt_cameras="$(arg pt_cameras)"/>
   <!-- ETV-CG Cameras -->
-  <xacro:etvcg_cameras parent="root"/>
+  <xacro:if value="$(arg etv_cg_cameras)">
+    <xacro:etvcg_cameras parent="root"/>
+  </xacro:if>
 </robot>

File: urdf/canadarm2.urdf.xacro (robot description, xacro)
@@ -3,5 +3,5 @@
   <xacro:include filename="$(find iss_description)/urdf/pt_camera.urdf.xacro"/>
   <xacro:include filename="$(find iss_description)/urdf/pt_camera.gazebo.xacro"/>
-  <xacro:macro name="canadarm2" params=" parent:='' ">
+  <xacro:macro name="canadarm2" params=" parent:='' pt_cameras:=True">
   <link name="pdgf"/>
   <link name="pdgf_forward"/>
@@ -222,26 +222,28 @@
       <limit effort="5000.0" lower="-3.1416" upper="3.1416" velocity="0.04"/>
   </joint>
-  <xacro:pt_camera prefix="boom_a_clpa" parent_link="canadarm2_link_3">
-    <origin xyz="-4.591 0.259 0.0" rpy="1.5708 0.0 1.5708"/>
-  </xacro:pt_camera>
-  <xacro:pt_camera_gazebo
-    prefix="boom_a_clpa"
-    image_width="1024"
-    image_height="1024"
-    horizontal_fov="0.896"
-    update_rate="30.0"
-    enable_lens_flare="true"
-    lens_flare_scale="5.0"/>
-  <xacro:pt_camera prefix="boom_b_clpa" parent_link="canadarm2_link_4">
-    <origin xyz="0.142 -0.847 2.735" rpy="0.0 0.0 0.0"/>
-  </xacro:pt_camera>
-  <xacro:pt_camera_gazebo
-    prefix="boom_b_clpa"
-    image_width="1024"
-    image_height="1024"
-    horizontal_fov="0.896"
-    update_rate="30.0"
-    enable_lens_flare="true"
-    lens_flare_scale="5.0"/>
+  <xacro:if value="${pt_cameras}">
+    <xacro:pt_camera prefix="boom_a_clpa" parent_link="canadarm2_link_3">
+      <origin xyz="-4.591 0.259 0.0" rpy="1.5708 0.0 1.5708"/>
+    </xacro:pt_camera>
+    <xacro:pt_camera_gazebo
+      prefix="boom_a_clpa"
+      image_width="1024"
+      image_height="1024"
+      horizontal_fov="0.896"
+      update_rate="30.0"
+      enable_lens_flare="true"
+      lens_flare_scale="5.0"/>
+    <xacro:pt_camera prefix="boom_b_clpa" parent_link="canadarm2_link_4">
+      <origin xyz="0.142 -0.847 2.735" rpy="0.0 0.0 0.0"/>
+    </xacro:pt_camera>
+    <xacro:pt_camera_gazebo
+      prefix="boom_b_clpa"
+      image_width="1024"
+      image_height="1024"
+      horizontal_fov="0.896"
+      update_rate="30.0"
+      enable_lens_flare="true"
+      lens_flare_scale="5.0"/>
+  </xacro:if>
  </xacro:macro>
 </robot>

File: urdf/dextre.urdf.xacro (robot description, xacro)
@@ -4,5 +4,5 @@
   <xacro:include filename="$(find iss_description)/urdf/pt_camera.gazebo.xacro"/>
   <!-- DEXTRE -->
-  <xacro:macro name="dextre" params=" parent:='' ">
+  <xacro:macro name="dextre" params=" parent:='' pt_cameras:=True">
   <!-- ******* Link Base *******  -->
   <link name="dextre_base">
@@ -462,28 +462,30 @@
       <limit effort="1000.0" lower="-3.1416" upper="3.1416" velocity="0.5"/>
   </joint>
-  <!-- Outrigger 1 CLPA Camera on tool_platform -->
-  <xacro:pt_camera prefix="outrigger_1_clpa" parent_link="dextre_tool_platform">
-    <origin xyz="1.368 0.300 0.314" rpy="1.5708 0.0 0.0"/>
-  </xacro:pt_camera>
-  <xacro:pt_camera_gazebo
-    prefix="outrigger_1_clpa"
-    image_width="1024"
-    image_height="1024"
-    horizontal_fov="0.896"
-    update_rate="30.0"
-    enable_lens_flare="true"
-    lens_flare_scale="5.0"/>
-  <!-- Outrigger 2 CLPA Camera on tool_platform -->
-  <xacro:pt_camera prefix="outrigger_2_clpa" parent_link="dextre_tool_platform">
-    <origin xyz="-1.368 0.300 0.314" rpy="1.5708 0.0 0.0"/>
-  </xacro:pt_camera>
-  <xacro:pt_camera_gazebo
-    prefix="outrigger_2_clpa"
-    image_width="1024"
-    image_height="1024"
-    horizontal_fov="0.896"
-    update_rate="30.0"
-    enable_lens_flare="true"
-    lens_flare_scale="5.0"/>
+  <xacro:if value="${pt_cameras}">
+    <!-- Outrigger 1 CLPA Camera on tool_platform -->
+    <xacro:pt_camera prefix="outrigger_1_clpa" parent_link="dextre_tool_platform">
+      <origin xyz="1.368 0.300 0.314" rpy="1.5708 0.0 0.0"/>
+    </xacro:pt_camera>
+    <xacro:pt_camera_gazebo
+      prefix="outrigger_1_clpa"
+      image_width="1024"
+      image_height="1024"
+      horizontal_fov="0.896"
+      update_rate="30.0"
+      enable_lens_flare="true"
+      lens_flare_scale="5.0"/>
+    <!-- Outrigger 2 CLPA Camera on tool_platform -->
+    <xacro:pt_camera prefix="outrigger_2_clpa" parent_link="dextre_tool_platform">
+      <origin xyz="-1.368 0.300 0.314" rpy="1.5708 0.0 0.0"/>
+    </xacro:pt_camera>
+    <xacro:pt_camera_gazebo
+      prefix="outrigger_2_clpa"
+      image_width="1024"
+      image_height="1024"
+      horizontal_fov="0.896"
+      update_rate="30.0"
+      enable_lens_flare="true"
+      lens_flare_scale="5.0"/>
+  </xacro:if>
   </xacro:macro>
 </robot>

File: urdf/mobile_servicing_system.gazebo.xacro (robot description, xacro)
@@ -6,5 +6,5 @@
   <xacro:include filename="$(find iss_description)/urdf/solar_panels.gazebo.xacro"/>
   <xacro:include filename="$(find iss_description)/urdf/pt_camera.gazebo.xacro"/>
-  <xacro:macro name="mobile_servicing_system_gazebo" params="command_interface:=position">
+  <xacro:macro name="mobile_servicing_system_gazebo" params="command_interface:=position pt_cameras:=True etv_cg_cameras:=True">
     <ros2_control name="GazeboSystem" type="system">
       <hardware>
@@ -16,12 +16,16 @@
       <xacro:solar_panels_ros2_control_joints command_interface="${command_interface}"/>
       <!-- Pan-Tilt Camera Joints -->
-      <xacro:pt_camera_ros2_control prefix="boom_a_clpa"/>
-      <xacro:pt_camera_ros2_control prefix="boom_b_clpa"/>
-      <xacro:pt_camera_ros2_control prefix="outrigger_1_clpa"/>
-      <xacro:pt_camera_ros2_control prefix="outrigger_2_clpa"/>
-      <xacro:pt_camera_ros2_control prefix="etvcg_cp3"/>
-      <xacro:pt_camera_ros2_control prefix="etvcg_cp8"/>
-      <xacro:pt_camera_ros2_control prefix="etvcg_cp9"/>
-      <xacro:pt_camera_ros2_control prefix="etvcg_cp13"/>
+      <xacro:if value="${pt_cameras}">
+        <xacro:pt_camera_ros2_control prefix="boom_a_clpa"/>
+        <xacro:pt_camera_ros2_control prefix="boom_b_clpa"/>
+        <xacro:pt_camera_ros2_control prefix="outrigger_1_clpa"/>
+        <xacro:pt_camera_ros2_control prefix="outrigger_2_clpa"/>
+      </xacro:if>
+      <xacro:if value="${etv_cg_cameras}">
+        <xacro:pt_camera_ros2_control prefix="etvcg_cp3"/>
+        <xacro:pt_camera_ros2_control prefix="etvcg_cp8"/>
+        <xacro:pt_camera_ros2_control prefix="etvcg_cp9"/>
+        <xacro:pt_camera_ros2_control prefix="etvcg_cp13"/>
+      </xacro:if>
     </ros2_control>
   <gazebo>

Commit message: Hotfix/add if cameras (#5)
* Added if simulate cameras to opt to simulate them or not

* fix launch error when using launch configruation in OnProcessExit scope

---------

Co-authored-by: Kenji Brameld <kbrameld@traclabs.com>

File: robots/mobile_servicing_system.urdf.xacro (robot description, xacro)
@@ -1,21 +1,9 @@
 <?xml version="1.0"?>
 <robot name="mobile_servicing_system" xmlns:xacro="http://www.ros.org/wiki/xacro">
-  <xacro:include filename="$(find iss_description)/urdf/mobile_base_system.urdf.xacro"/>
-  <xacro:include filename="$(find iss_description)/urdf/canadarm2.urdf.xacro"/>
-  <xacro:include filename="$(find iss_description)/urdf/dextre.urdf.xacro"/>
-  <xacro:include filename="$(find iss_description)/urdf/solar_panels.urdf.xacro"/>
-  <xacro:include filename="$(find iss_description)/urdf/etvcg_cameras.urdf.xacro"/>
-  <!-- Gazebo -->
-  <xacro:include filename="$(find iss_description)/urdf/mobile_servicing_system.gazebo.xacro"/>
-  <xacro:mobile_servicing_system_gazebo command_interface="position"/>
-  <!-- ISS and Mobile Base System -->
-  <link name="world"/>
-  <xacro:mobile_base_system parent="world"/>
-  <!-- Solar Panels -->
-  <xacro:solar_panels parent="link_14_s0_truss"/>
-  <!-- Canadarm2 and Dextre -->
-  <xacro:dextre parent="canadarm2_link_7"/>
-  <xacro:canadarm2 parent="mobile_base_system"/>
-  <!-- ETV-CG Cameras -->
-  <xacro:etvcg_cameras parent="root"/>
+  <xacro:include filename="$(find iss_description)/urdf/mobile_servicing_system.macro.xacro"/>
+  <xacro:arg name="etv_cg_cameras" default="True"/>
+  <xacro:arg name="pt_cameras" default="True"/>
+  <xacro:mobile_servicing_system etv_cg_cameras="$(arg etv_cg_cameras)"
+                                 pt_cameras="$(arg pt_cameras)">
+  </xacro:mobile_servicing_system>
 </robot>
